File: hw/Lab_6.brd (EAGLE design)
At the start: 131.1 x 89.1 mm, 36 parts, among them U1 TM4C123GH6PM, U2 LP2950-3.3ACZ, U3 LM4041CILPRCLP, Y1 16MHZ_CRYSTAL

Commit message: Final PCB design
Requirement Document fulfilled
Parts:
- removed U3: LM4041CILPRCLP, EE445L:LP_O-PBCY-W3
- added C16, C17: 0.1uf, EE445L:CAP100MIL
- added DAC: AD8300ARZ, AD8300ARZ:SOIC127P600X175-8N
- added OPAMP: RC4558D, RC4558D:SOIC127P600X175-8N
- added R5: 1K, EE445L:RES200MIL
- R4: value (none) -> 10K
- moved R4 139.4 mm to (122.5, 29.4), flipped to the bottom, turned to 90 degrees
- moved R2 127.2 mm to (111.6, 51.2), turned to 180 degrees
- moved LED1 126.9 mm to (101.2, 36.1), flipped to the bottom, turned to 270 degrees
- moved RESET 119.3 mm to (109.9, 43.5), flipped to the bottom, turned to 90 degrees
- moved R3 95.5 mm to (89.1, 52.0)
- moved JP5 80.5 mm to (40.4, 21.2), flipped to the bottom
- moved 3.7V 78.7 mm to (38.9, 37.0), turned to 180 degrees
- moved JP2 75.7 mm to (40.4, 32.1), flipped to the bottom
- moved JP6 70.1 mm to (40.4, 27.4), flipped to the bottom, turned to 180 degrees
- moved U2 63.2 mm to (25.3, 29.7), turned to 90 degrees
- moved LED2 52.2 mm to (27.8, 22.7), flipped to the bottom
- moved C13 52.0 mm to (25.9, 36.4), turned to 180 degrees
- moved GND1 51.1 mm to (12.1, 6.55)
- moved C15 44.6 mm to (109.7, 36.2), turned to 180 degrees
- moved C14 42.4 mm to (13.7, 34.5), turned to 180 degrees
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Connections:
- new net ANALOGOUT: JP4.1, OPAMP.1, OPAMP.2
- new net LEDVOLTAGE: LED1.A, R5.1
- new net PD0: DAC.3, JP3.9, U1.61
- new net PD1: DAC.2, JP3.7, U1.62
- new net PD3: DAC.4, JP3.5, U1.64
- new net PD6: DAC.5, JP3.3, U1.53
- new net PD7: DAC.6, JP3.1, U1.10
- new net PE2: R4.2, U1.7
- new net PE3: JP3.15, U1.6
- new net PE4: JP3.13, MODE.3, MODE.4, U1.59
- new net PE5: JP3.11, R5.2, U1.60
- new net VOUT: DAC.8, OPAMP.3
- net +3V3: now also C16.1, C17.1, DAC.1, MODE.1, MODE.2, OPAMP.8, R4.1
- net GND: now also C16.2, C17.2, DAC.7, JP4.2, LED1.K, OPAMP.4, R4.3
Routing:
- net GND: track 49.8 -> 508.2 mm, vias 6 -> 15
- net +3V3: track 29.6 -> 390.5 mm, vias 0 -> 6
- net PE4: track 0.00 -> 150.4 mm, vias 0 -> 5
- net PE5: track 0.00 -> 129.5 mm, vias 0 -> 4
- net PD0: track 0.00 -> 104.9 mm, vias 0 -> 4
- net PD1: track 0.00 -> 104.4 mm, vias 0 -> 5
- net PD7: track 0.00 -> 104.3 mm, vias 0 -> 6
- net PD3: track 0.00 -> 101.0 mm, vias 0 -> 3
- net PE3: track 0.00 -> 81.2 mm, vias 0 -> 4
- net PD6: track 0.00 -> 77.3 mm, vias 0 -> 4
- net PE2: track 0.00 -> 65.9 mm, vias 0 -> 2
- net RESET: track 0.00 -> 60.6 mm, vias 0 -> 2
- net VOUT: track 0.00 -> 34.4 mm, vias 0 -> 2
- net WAKE: track 0.00 -> 23.9 mm, vias 0 -> 1
- net +3.7V: track 0.00 -> 22.4 mm
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Other:
- board size 131.1 x 89.1 mm -> 128.5 x 72.4 mm
- board text added: "GND"
- board text added: "Marzooq Shah Lab 6 ECE445L"
- board text added: "TA: Jared McArthur"
- board text added: "TCK"
- board text added: "TDI"
- board text added: "TDO"
- board text added: "TMS"
